Commit message: Joint name changes

File: my_robot/urdf/my_robot.xacro (robot description, xacro)
@@ -59,5 +59,5 @@
   </link>
 	<!-- LEFT DRIVE -->
-  <joint type="continuous" name="left_drive">
+  <joint type="continuous" name="left_drive_joint">
     <origin xyz="0 0.15 0" rpy="0 0 0"/>
     <child link="left_drive"/>
@@ -91,5 +91,5 @@
   </link>
 	<!-- RIGHT DRIVE -->
-  <joint type="continuous" name="right_drive">
+  <joint type="continuous" name="right_drive_joint">
     <origin xyz="0 -0.15 0" rpy="0 0 0"/>
     <child link="right_drive"/>
